File: Endgame/EndgameV2.sch (KiCad schematic (older format))
At the start: 158 parts, among them J1 OLED, SW1 Rotary_Encoder, SW2 SW_PUSH, U1 ATmega32U4-AU, U2 ai03-locallib_PRTR5V0U2X, Y1 Crystal_GND24_Small

Commit message: Add resistor to RST
Parts:
- added R?: 10k, Resistor_SMD:R_0805_2012Metric, symbol Device:R_Small
- C3, C5, C6, C7, C8: symbol keyboard_parts:C -> EndgameV2-rescue:C-keyboard_parts
- J1: symbol oled:OLED -> EndgameV2-rescue:OLED-oled
- R7, R8, R9: symbol keyboard_parts:R -> EndgameV2-rescue:R-keyboard_parts
- SW2: symbol keyboard_parts:SW_PUSH -> EndgameV2-rescue:SW_PUSH-keyboard_parts
- S_"1, S_+1, S_,1, S_-1, S_.1, S_0, S_1, S_10, S_2, S_3, S_4, S_5, S_6, S_7, S_8, S_9, S_;1, S_A1, S_B1, S_BkSp1, S_C1, S_Cap_Lk1, S_D1, S_DOWN1, S_Del1, S_E1, S_Ent1, S_Esc1, S_F1, S_For_Slash1, S_G1, S_H1, S_I1, S_Ins1, S_J1, S_K1, S_L1, S_LEFT1, S_L_ALT1, S_L_CTRL1, S_L_Shift1, S_L_WIN1, S_M1, S_N1, S_O1, S_P1, S_Pg_Dn1, S_Pg_Up1, S_Q1, S_R1, S_RIGHT1, S_R_ALT1, S_R_CTRL1, S_R_FN1, S_R_Shift1, S_S1, S_SPACE1, S_T1, S_Tab1, S_U1, S_UP1, S_V1, S_W1, S_X1, S_Y1, S_Z1, S_[1, S_]1: symbol MX_Alps_Hybrid:MX-NoLED -> EndgameV2-rescue:MX-NoLED-MX_Alps_Hybrid
- U1: symbol MCU_Microchip_ATmega:ATmega32U4-AU -> EndgameV2-rescue:ATmega32U4-AU-MCU_Microchip_ATmega
- U2: symbol cpm43-cache:ai03-locallib_PRTR5V0U2X -> EndgameV2-rescue:ai03-locallib_PRTR5V0U2X-cpm43-cache
- USB1: symbol cpm43-cache:Type-C_HRO-TYPE-C-31-M-12 -> EndgameV2-rescue:Type-C_HRO-TYPE-C-31-M-12-cpm43-cache
Connections:
- net +5V: now also R?.2
- net at SW2.2, U1.13 (~RESET): now also R?.1

Commit message: Added ISCP
Parts:
- added J?: AVR-ISP-6, symbol Connector:AVR-ISP-6
Connections:
- net +5V: now also J?.2 (VCC)
- net EN1: now also U1.1 (PE6); no longer U1.11 (PB3)
- net EN2: now also U1.12 (PB7); no longer U1.10 (PB2)
- net GND: now also J?.6 (GND)
- net RST: now reaches R?.1, SW2.2, U1.13 (~RESET)
- net RST: now also J?.5 (~RST)
- net SCK: now reaches U1.9 (PB1)
- net SCK: now also J?.3 (SCK)
- new net MISO: J?.1 (MISO), U1.11 (PB3)
- new net MOSI: J?.4 (MOSI), U1.10 (PB2)
Other:
- moved on the sheet: J1
Changed lines of the file:
@@
 Text GLabel 4500 900  1    50   Input ~ 0
 COL1
-Text GLabel 3400 1600 0    50   Input ~ 0
+Text GLabel 3400 1600 1    50   Input ~ 0
 ROW0
-Text GLabel 3400 2250 0    50   Input ~ 0
+Text GLabel 3400 2250 1    50   Input ~ 0
 ROW1
-Text GLabel 3400 2900 0    50   Input ~ 0
+Text GLabel 3400 2900 1    50   Input ~ 0
 ROW2
-Text GLabel 3400 3550 0    50   Input ~ 0
+Text GLabel 3400 3550 1    50   Input ~ 0
 ROW3
-Text GLabel 3400 4200 0    50   Input ~ 0
+Text GLabel 3400 4200 1    50   Input ~ 0
 ROW4
 Text GLabel 5000 900  1    50   Input ~ 0
@@
 L EndgameV2-rescue:OLED-oled J1
 U 1 1 5DD5B4B8
-P 8700 4850
-F 0 "J1" H 8617 4475 50  0000 C CNN
-F 1 "OLED" H 8617 4566 50  0000 C CNN
-F 2 "Lily58-footprint:OLED_4Pin" H 8700 4850 50  0001 C CNN
-F 3 "" H 8700 4850 50  0000 C CNN
-	1    8700 4850
-	1    0    0    -1
-$EndComp
-Wire Wire Line
-	8500 4700 8250 4700
+P 10900 6050
+F 0 "J1" H 10817 5675 50  0000 C CNN
+F 1 "OLED" H 10817 5766 50  0000 C CNN
+F 2 "Lily58-footprint:OLED_4Pin" H 10900 6050 50  0001 C CNN
+F 3 "" H 10900 6050 50  0000 C CNN
+	1    10900 6050
+	1    0    0    -1
+$EndComp
+Wire Wire Line
+	10700 5900 10450 5900
 $Comp
 L EndgameV2-rescue:GND-gnd #PWR0116
 U 1 1 5DDA38A1
-P 8250 4700
-F 0 "#PWR0116" H 8250 4450 50  0001 C CNN
-F 1 "GND" H 8250 4789 50  0000 C CNN
-F 2 "" H 8250 4700 50  0001 C CNN
-F 3 "" H 8250 4700 50  0001 C CNN
-	1    8250 4700
-	1    0    0    -1
-$EndComp
-Text GLabel 8500 4900 0    50   Input ~ 0
+P 10450 5900
+F 0 "#PWR0116" H 10450 5650 50  0001 C CNN
+F 1 "GND" H 10450 5989 50  0000 C CNN
+F 2 "" H 10450 5900 50  0001 C CNN
+F 3 "" H 10450 5900 50  0001 C CNN
+	1    10450 5900
+	1    0    0    -1
+$EndComp
+Text GLabel 10700 6100 0    50   Input ~ 0
 SCL
-Text GLabel 8500 5000 0    50   Input ~ 0
+Text GLabel 10700 6200 0    50   Input ~ 0
 SDA
 Wire Wire Line
@@
 Text GLabel 2950 6050 2    50   Input ~ 0
 COL10
-Text GLabel 2950 3550 2    50   Input ~ 0
+Text GLabel 2950 5450 2    50   Input ~ 0
 EN1
-Text GLabel 2950 3450 2    50   Input ~ 0
+Text GLabel 2950 3950 2    50   Input ~ 0
 EN2
 Text GLabel 2950 5050 2    50   Input ~ 0
@@
 L power:+5V #PWR?
 U 1 1 5DF42376
-P 8100 4800
-F 0 "#PWR?" H 8100 4650 50  0001 C CNN
-F 1 "+5V" H 8115 4973 50  0000 C CNN
-F 2 "" H 8100 4800 50  0001 C CNN
-F 3 "" H 8100 4800 50  0001 C CNN
-	1    8100 4800
-	1    0    0    -1
-$EndComp
-Wire Wire Line
-	8100 4800 8500 4800
+P 10300 6000
+F 0 "#PWR?" H 10300 5850 50  0001 C CNN
+F 1 "+5V" H 10315 6173 50  0000 C CNN
+F 2 "" H 10300 6000 50  0001 C CNN
+F 3 "" H 10300 6000 50  0001 C CNN
+	1    10300 6000
+	1    0    0    -1
+$EndComp
+Wire Wire Line
+	10300 6000 10700 6000
 $Comp
 L Device:R_Small R?
@@
 Wire Wire Line
 	1500 2900 1500 2750
+$Comp
+L Connector:AVR-ISP-6 J?
+U 1 1 5DF23484
+P 9400 5100
+F 0 "J?" H 9071 5196 50  0000 R CNN
+F 1 "AVR-ISP-6" H 9071 5105 50  0000 R CNN
+F 2 "" V 9150 5150 50  0001 C CNN
+F 3 " ~" H 8125 4550 50  0001 C CNN
+	1    9400 5100
+	1    0    0    -1
+$EndComp
+Text GLabel 9800 4900 2    50   Input ~ 0
+MISO
+Text GLabel 9800 5000 2    50   Input ~ 0
+MOSI
+Text GLabel 9800 5100 2    50   Input ~ 0
+SCK
+Text GLabel 9800 5200 2    50   Input ~ 0
+RST
+$Comp
+L power:+5V #PWR?
+U 1 1 5DF4285F
+P 9300 4600
+F 0 "#PWR?" H 9300 4450 50  0001 C CNN
+F 1 "+5V" H 9315 4773 50  0000 C CNN
+F 2 "" H 9300 4600 50  0001 C CNN
+F 3 "" H 9300 4600 50  0001 C CNN
+	1    9300 4600
+	1    0    0    -1
+$EndComp
+$Comp
+L power:GND #PWR?
+U 1 1 5DF44397
+P 9300 5500
+F 0 "#PWR?" H 9300 5250 50  0001 C CNN
+F 1 "GND" H 9305 5327 50  0000 C CNN
+F 2 "" H 9300 5500 50  0001 C CNN
+F 3 "" H 9300 5500 50  0001 C CNN
+	1    9300 5500
+	1    0    0    -1
+$EndComp
+Text GLabel 2950 3350 2    50   Input ~ 0
+SCK
+Text GLabel 2950 3450 2    50   Input ~ 0
+MOSI
+Text GLabel 2950 3550 2    50   Input ~ 0
+MISO
+Text GLabel 1350 3250 1    50   Input ~ 0
+RST
 $EndSCHEMATC
